File: hardware/IR_Termostat/IR_Termostat.kicad_pcb (KiCad board)
At the start: 2 copper layers, 14 parts, among them J1 USB_C_Receptacle_PowerOnly_6P, Q1 PMOS, U1 TP4056-42-ESOP8, U2 XC6206PxxxMR

Commit message: Fix: power path mosfet footprint
 The footprint of the power path mosfet now it's pin-to-pin with the skemathic.
Parts:
- added C4: 100nF 16V, Capacitor_SMD:C_0805_2012Metric_Pad1.18x1.45mm_HandSolder, F.Cu at (126.8, 86.9)
- added C5: 10uF 16V, Capacitor_SMD:C_0805_2012Metric_Pad1.18x1.45mm_HandSolder, F.Cu at (126.8, 89.9)
- added C6: 100nF 16V, Capacitor_SMD:C_0805_2012Metric_Pad1.18x1.45mm_HandSolder, F.Cu at (126.8, 92.9)
- added C7: 100nF 16V, Capacitor_SMD:C_0805_2012Metric_Pad1.18x1.45mm_HandSolder, F.Cu at (126.8, 95.9)
- added C8: 100nF 16V, Capacitor_SMD:C_0805_2012Metric_Pad1.18x1.45mm_HandSolder, F.Cu at (126.8, 98.9)
- added D2: BZT52C4V7, Diode_SMD:D_SOD-123F, F.Cu at (149.6, 110.0)
- added J2: JST-PH-2mm, Connector_JST:JST_PH_S2B-PH-K_1x02_P2.00mm_Horizontal, F.Cu at (146.4, 87.8)
- added LDR1: GL5516, OptoDevice:R_LDR_5.1x4.3mm_P3.4mm_Vertical, F.Cu at (148.5, 100.0)
- added R10: 10K 1%, Resistor_SMD:R_0805_2012Metric_Pad1.20x1.40mm_HandSolder, F.Cu at (136.3, 89.8)
- added R11: 22K 1%, Resistor_SMD:R_0805_2012Metric_Pad1.20x1.40mm_HandSolder, F.Cu at (136.3, 92.8)
- added R12: 9.1K 1%, Resistor_SMD:R_0805_2012Metric_Pad1.20x1.40mm_HandSolder, F.Cu at (136.3, 95.7)
- added R13: 1K 1%, Resistor_SMD:R_0805_2012Metric_Pad1.20x1.40mm_HandSolder, F.Cu at (141.1, 86.8)
- added R14: 5.1K 1%, Resistor_SMD:R_0805_2012Metric_Pad1.20x1.40mm_HandSolder, F.Cu at (141.1, 89.8)
- added R15: 5.1K 1%, Resistor_SMD:R_0805_2012Metric_Pad1.20x1.40mm_HandSolder, F.Cu at (141.1, 92.8)
- added R16: 22K 1%, Resistor_SMD:R_0805_2012Metric_Pad1.20x1.40mm_HandSolder, F.Cu at (141.1, 95.7)
- added R5: 22K 1%, Resistor_SMD:R_0805_2012Metric_Pad1.20x1.40mm_HandSolder, F.Cu at (131.6, 86.8)
- added R6: 1K 1%, Resistor_SMD:R_0805_2012Metric_Pad1.20x1.40mm_HandSolder, F.Cu at (131.6, 89.8)
- added R7: 10K 1%, Resistor_SMD:R_0805_2012Metric_Pad1.20x1.40mm_HandSolder, F.Cu at (131.6, 92.8)
- added R8: 10K 1%, Resistor_SMD:R_0805_2012Metric_Pad1.20x1.40mm_HandSolder, F.Cu at (131.6, 95.7)
- added R9: 1K 1%, Resistor_SMD:R_0805_2012Metric_Pad1.20x1.40mm_HandSolder, F.Cu at (136.3, 86.8)
- added SW1: SW_Push_Dual, Button_Switch_SMD:SW_SPST_CK_KMS2xxGP, F.Cu at (150.1, 105.4)
- added TV1: PESD5V0S1BA, Diode_SMD:D_SOD-323_HandSoldering, F.Cu at (143.2, 76.0)
- added U3: ~, Package_SO:SOIC-8-1EP_3.9x4.9mm_P1.27mm_EP2.29x3mm_ThermalVias, F.Cu at (133.4, 100.5)
- added U4: MLX90614ESF-BAA-000-TU, Library:TO254P942H425-4, F.Cu at (139.0, 60.5)
- added U5: CH32V003JxMx, Package_SO:SOP-8_3.9x4.9mm_P1.27mm, F.Cu at (133.4, 107.1)
- added U6: DM-OLED096-636, Library:MODULE_DM-OLED096-636, F.Cu at (163.5, 63.0)
- Q1: value PMOS -> FDN306P; footprint Package_TO_SOT_SMD:SOT-23_Handsoldering -> Package_TO_SOT_SMD:SOT-23
- U2: value XC6206PxxxMR -> XC6206P-3.3V
- moved J1 83.0 mm to (168.6, 85.2)
- moved C1 82.7 mm to (176.5, 89.5)
- moved C3 82.7 mm to (176.5, 95.5)
- moved Q1 82.7 mm to (190.0, 102.5)
- moved R1 82.7 mm to (159.9, 89.5)
- moved R2 82.7 mm to (159.9, 92.4)
- moved R4 82.7 mm to (159.9, 98.3)
- moved TH1 82.7 mm to (159.9, 101.2)
- moved C2 82.7 mm to (176.5, 92.5)
- moved D1 82.7 mm to (175.8, 104.2)
- moved R3 82.7 mm to (159.9, 95.3)
- moved U1 82.7 mm to (166.5, 100.6)
- moved U2 82.7 mm to (173.3, 99.7)
- moved F1 82.7 mm to (173.7, 108.1)
Connections:
- net Net-(U2-VO) renamed +3.3V
- C2 pad 2: Net-(U2-GND) -> GND
- C3 pad 2: Net-(U2-GND) -> GND
- Q1 pad 1: unconnected-(Q1-D-Pad1) -> +5V
- Q1 pad 2: unconnected-(Q1-G-Pad2) -> Net-(D1-K)
- Q1 pad 3: unconnected-(Q1-S-Pad3) -> Vbat+
- U1 pad 6: unconnected-(U1-~{STDBY}-Pad6) -> STDBY
- U1 pad 7: unconnected-(U1-~{CHRG}-Pad7) -> CHRG
- U2 pad 1: Net-(U2-GND) -> GND
