File: hardware/IR_Termostat/IR_Termostat.kicad_pcb (KiCad board)
At the start: 2 copper layers, 40 parts, among them J1 USB_C_Receptacle_PowerOnly_6P, J2 JST-PH-2mm, Q1 FDN306P, SW1 SW_Push_Dual, U1 TP4056-42-ESOP8, U2 XC6206P-3.3V, U4 MLX90614ESF-BAA-000-TU, U5 CH32V003JxMx, U6 DM-OLED096-636

Commit message: Feat: First components layout
Parts:
- removed U6: DM-OLED096-636, Library:MODULE_DM-OLED096-636
- added DISPLAY_1: DM-OLED096-636, Library:MODULE_DM-OLED096-636, F.Cu at (152.5, 85.0)
- added J3: Conn_01x03_Pin, Connector_PinHeader_2.54mm:PinHeader_1x03_P2.54mm_Vertical, F.Cu at (146.0, 109.5)
- C7, C8, J2, U4: moved to B.Cu
- SW1: value SW_Push_Dual -> SW_SPST; footprint Button_Switch_SMD:SW_SPST_CK_KMS2xxGP -> Button_Switch_THT:SW_PUSH_6mm
- moved J1 48.0 mm to (153.5, 130.7)
- moved C4 47.7 mm to (158.5, 122.5), turned to -90 degrees
- moved TV1 47.5 mm to (146.5, 123.4), turned to -90 degrees
- moved C1 47.4 mm to (143.5, 123.5), turned to 180 degrees
- moved C5 45.2 mm to (156.5, 124.0), turned to -90 degrees
- moved R1 43.8 mm to (138.7, 127.7), turned to -90 degrees
- moved R6 39.5 mm to (153.0, 123.0), turned to 180 degrees
- moved J2 38.2 mm to (152.0, 125.5)
- moved U3 36.8 mm to (163.3, 122.0), turned to 180 degrees
- moved R11 36.5 mm to (167.0, 112.5), turned to -90 degrees
- moved U1 35.9 mm to (143.5, 128.2)
- moved Q1 34.7 mm to (158.4, 117.0), turned to 90 degrees
- moved C3 34.3 mm to (153.0, 120.5), turned to 180 degrees
- moved R5 33.1 mm to (149.0, 115.0), turned to 90 degrees
- moved C8 33.0 mm to (150.0, 75.5), turned to 180 degrees
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Connections:
- Q1 pad 2: Net-(D1-K) -> Vbat+
- Q1 pad 3: Vbat+ -> Net-(D1-K)
- TV1 pad 1: unconnected-(TV1-A-Pad1) -> GND
- U1 pad 6: STDBY -> unconnected-(U1-~{STDBY}-Pad6)
Other:
- board outline added: 30.5 x 63 mm

Commit message: feat: first pcb v0.1
Parts:
- removed R8: 10K 1%, Resistor_SMD:R_0805_2012Metric_Pad1.20x1.40mm_HandSolder
- moved R10 22.2 mm to (166.0, 103.5), turned to 90 degrees
- moved R11 7.21 mm to (161.0, 108.5), turned to 180 degrees
- moved C7 7.11 mm to (151.5, 86.0), turned to 180 degrees
- moved R15 5.65 mm to (140.5, 99.5), turned to 90 degrees
- moved R14 4.17 mm to (142.5, 99.5), turned to 90 degrees
- moved R2 3.03 mm to (139.9, 121.6), turned to 180 degrees
- moved C5 2.00 mm to (156.5, 122.0)
- moved DISPLAY_1 1.50 mm to (152.5, 83.5)
- moved C8 1.46 mm to (150.0, 74.0)
- moved U4 0.92 mm to (153.0, 80.0), turned to -90 degrees
- moved U1 0.81 mm to (144.3, 128.3)
- moved R1 0.80 mm to (139.5, 127.7)
- moved C4 0.57 mm to (158.5, 122.0)
- moved J2 0.55 mm to (152.0, 125.0)
- moved R12 0.50 mm to (165.0, 108.5), turned to 180 degrees
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Routing:
- net +3.3V: track 0.00 -> 115.1 mm
- net GND: track 0.00 -> 113.3 mm, vias 0 -> 17
- net +5V: track 0.00 -> 61.1 mm, vias 0 -> 2
- net SCL: track 0.00 -> 44.9 mm
- net SDA: track 0.00 -> 43.4 mm
- net Vbat+: track 0.00 -> 29.7 mm, vias 0 -> 1
- net CHRG: track 0.00 -> 28.5 mm, vias 0 -> 4
- net Net-(U5-PA2): track 0.00 -> 20.1 mm
- net SWIO: track 0.00 -> 17.1 mm
- net Net-(U5-PD6/PA1): track 0.00 -> 16.7 mm
- net Net-(J2-Pin_2): track 0.00 -> 16.7 mm
- net Net-(D1-K): track 0.00 -> 12.4 mm
- net Net-(J1-CC2): track 0.00 -> 10.4 mm
- net Net-(SW1-A): track 0.00 -> 9.91 mm
- net Net-(F1-Pad1): track 0.00 -> 9.63 mm
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- added copper zone on B.Cu, net GND
Other:
- board size 30.5 x 63 mm -> 30.5 x 64.5 mm
- board text added: "BATTERY"
- board text added: "Termostat v0.1"
